Commit message: 1

File: robarm_ws/src/my_bot/config/robarm.ros2_control.xacro (robot description, xacro)
@@ -14,5 +14,7 @@
                 </state_interface>
                 <state_interface name="velocity"/>
-            </joint>
+            <dynamics damping="0.05" friction="0.08"/>
+    <dynamics damping="0.05" friction="0.08"/>
+    </joint>
             <joint name="arm_joint2">
                 <command_interface name="position"/>
@@ -21,5 +23,6 @@
                 </state_interface>
                 <state_interface name="velocity"/>
-            </joint>
+            <dynamics damping="0.05" friction="0.08"/>
+    </joint>
             <joint name="arm_joint3">
                 <command_interface name="position"/>
@@ -28,5 +31,6 @@
                 </state_interface>
                 <state_interface name="velocity"/>
-            </joint>
+            <dynamics damping="0.05" friction="0.08"/>
+    </joint>
             <joint name="arm_joint4">
                 <command_interface name="position"/>
@@ -35,5 +39,6 @@
                 </state_interface>
                 <state_interface name="velocity"/>
-            </joint>
+            <dynamics damping="0.05" friction="0.08"/>
+    </joint>
             <joint name="arm_joint5">
                 <command_interface name="position"/>
@@ -42,5 +47,6 @@
                 </state_interface>
                 <state_interface name="velocity"/>
-            </joint>
+            <dynamics damping="0.05" friction="0.08"/>
+    </joint>
             <joint name="grip_joint">
                 <command_interface name="position"/>
@@ -49,5 +55,6 @@
                 </state_interface>
                 <state_interface name="velocity"/>
-            </joint>
+            <dynamics damping="0.05" friction="0.08"/>
+    </joint>
         </ros2_control>
     </xacro:macro>

File: robarm_ws/src/rob_arm_info/urdf/robarm.urdf (robot description, URDF)
Before this commit: robot robarm, 12 links, 11 joints
Links:
- added link world
- link base_link: mass None -> 1.5
Joints:
- added joint world_fixed_joint: type fixed, parent world, child base_link, origin xyz=0 0 0 rpy=0 0 0
